File: commodorelcd.kicad_sch (KiCad schematic)
At the start: 236 parts, among them CN1 Conn_02x25_Odd_Even, CN11 Memory Board, CN2 DB37_Female_MountingHoles, CN3 Conn_02x13_Odd_Even, CN4 DB9_Female, CN5 Ext, CN6 Line, CN7 CBM Serial, CN9 LCD Panel, J1 Barrel_Jack_Switch, Q10 Q_PNP_BCE, Q11 Q_PNP_BCE, Q13 VN2222L, Q14 VP0300L, Q15 VN2222L, Q16 Q_PNP_BCE, Q17 VP0300L, Q19 Q_PNP_BCE, Q20 Q_NPN_BCE, Q5 VP0300L, Q8 Q_PNP_BCE, Q9 Q_PNP_BCE, SW1 Reset, SW2 NMI, SW3 SW_QPDT_Split, T1 L_Iron_Coupled_1243, U1 65102, U10 LM324, U11 4N28, U12 74HC14, U13 74HC244, U14 74HC245, U15 74HC374, U16 27C64, U17 74HC14, U18 LP365, U19 74HC165, U2 5707, U20 74HC165, U22 74HC02, U23 LM358, U24 74LS157, U25 74HC32, U26 74HC139, U3 5706, U4 6522, U5 6522, U6 6551, U7 S3530, U8 MSM58321RS, U9 74HC374, Y1 4MHz, Y2 1.8432 MHz, Y3 3.579545 MHz, Y5 32.768k

Commit message: Fix component references
Parts:
- L1: renamed from L?; value L_Iron -> 37 µH
- U31: renamed from U?; value TLP3546 -> LCA110
- gave numbers to parts that had none: 14
Connections:
- net ~{RAM1_CS}: no longer U28.20 (~{CS1}), U29.20 (~{CS1}), U30.20 (~{CS1})
- net ~{RAM2_CS}: now also U28.20 (~{CS1})
- net ~{RAM3_CS}: now also U29.20 (~{CS1})
- net ~{RAM4_CS}: now also U30.20 (~{CS1})
- net at CR2.1 (K), CR3.1 (K), R16.2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: now also U31.4
Other:
- moved on the sheet: C10, C34, C36, C51, C63, R53, R54, U10E, U12A, U23C, U31
